File: Evangelion_Unidad_00/Evangelion_Unidad_00.kicad_sch (KiCad schematic)
At the start: 2 parts, among them J1 CONN_01X11, U1 BluePill

Commit message: new
Parts:
- removed U1: BluePill, EESTN5:BluePill_2, symbol EESTN5:BluePill

Commit message: new
Parts:
- added U1: ESP32_DevKit_V1_DOIT, ESP32_DevKit_V1_DOIT:esp32_devkit_v1_doit, symbol EESTN5:ESP32_DevKit_V1_DOIT
Changed lines of the file:
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@@
 (kicad_sch
-	(version 20231120)
+	(version 20250114)
 	(generator "eeschema")
-	(generator_version "8.0")
+	(generator_version "9.0")
 	(paper "A4")
 	(junction
@@
 	(label "D2"
 		(at 236.22 64.77 180)
-		(fields_autoplaced yes)
 		(effects
 			(font
@@
 	(label "D5"
 		(at 227.33 92.71 0)
-		(fields_autoplaced yes)
 		(effects
 			(font
@@
 	(label "IR"
 		(at 227.33 105.41 0)
-		(fields_autoplaced yes)
 		(effects
 			(font
@@
 	(label "D7"
 		(at 227.33 87.63 0)
-		(fields_autoplaced yes)
 		(effects
 			(font
@@
 	(label "D3"
 		(at 227.33 97.79 0)
-		(fields_autoplaced yes)
 		(effects
 			(font
@@
 	(label "D3"
 		(at 236.22 62.23 180)
-		(fields_autoplaced yes)
 		(effects
 			(font
@@
 	(label "D1"
 		(at 227.33 102.87 0)
-		(fields_autoplaced yes)
 		(effects
 			(font
@@
 	(label "D5"
 		(at 236.22 57.15 180)
-		(fields_autoplaced yes)
 		(effects
 			(font
@@
 	(label "D6"
 		(at 236.22 54.61 180)
-		(fields_autoplaced yes)
 		(effects
 			(font
@@
 	(label "D4"
 		(at 236.22 59.69 180)
-		(fields_autoplaced yes)
 		(effects
 			(font
@@
 	(label "D7"
 		(at 236.22 52.07 180)
-		(fields_autoplaced yes)
 		(effects
 			(font
@@
 	(label "D2"
 		(at 227.33 100.33 0)
-		(fields_autoplaced yes)
 		(effects
 			(font
@@
 	(label "D1"
 		(at 236.22 67.31 180)
-		(fields_autoplaced yes)
 		(effects
 			(font
@@
 	(label "D8"
 		(at 227.33 85.09 0)
-		(fields_autoplaced yes)
 		(effects
 			(font
@@
 	(label "D6"
 		(at 227.33 90.17 0)
-		(fields_autoplaced yes)
 		(effects
 			(font
@@
 	(label "D4"
 		(at 227.33 95.25 0)
-		(fields_autoplaced yes)
 		(effects
 			(font
@@
 	(label "D8"
 		(at 236.22 49.53 180)
-		(fields_autoplaced yes)
 		(effects
 			(font
@@
 	)
 	(symbol
+		(lib_id "EESTN5:ESP32_DevKit_V1_DOIT")
+		(at 157.48 102.87 0)
+		(unit 1)
+		(exclude_from_sim no)
+		(in_bom yes)
+		(on_board yes)
+		(dnp no)
+		(fields_autoplaced yes)
+		(property "Reference" "U1"
+			(at 157.48 66.04 0)
+			(effects
+				(font
+					(size 1.27 1.27)
+				)
+			)
+		)
+		(property "Value" "ESP32_DevKit_V1_DOIT"
+			(at 157.48 68.58 0)
+			(effects
+				(font
+					(size 1.27 1.27)
+				)
+			)
+		)
+		(property "Footprint" "ESP32_DevKit_V1_DOIT:esp32_devkit_v1_doit"
+			(at 146.05 68.58 0)
+			(effects
+				(font
+					(size 1.27 1.27)
+				)
+				(hide yes)
+			)
+		)
+		(property "Datasheet" ""
+			(at 146.05 68.58 0)
+			(effects
+				(font
+					(size 1.27 1.27)
+				)
+				(hide yes)
+			)
+		)
+		(property "Description" ""
+			(at 157.48 102.87 0)
+			(effects
+				(font
+					(size 1.27 1.27)
+				)
+				(hide yes)
+			)
+		)
+		(pin "17"
+		)
+		(pin "1"
+		)
+		(pin "18"
+		)
+		(pin "8"
+		)
+		(pin "12"
+		)
+		(pin "28"
+		)
+		(pin "22"
+		)
+		(pin "3"
+		)
+		(pin "32"
+		)
+		(pin "2"
+		)
+		(pin "5"
+		)
+		(pin "4"
+		)
+		(pin "13"
+		)
+		(pin "33"
+		)
+		(pin "10"
+		)
+		(pin "15"
+		)
+		(pin "31"
+		)
+		(pin "30"
+		)
+		(pin "9"
+		)
+		(pin "11"
+		)
+		(pin "29"
+		)
+		(pin "27"
+		)
+		(pin "34"
+		)
+		(pin "36"
+		)
+		(pin "26"
+		)
+		(pin "35"
+		)
+		(pin "25"
+		)
+		(pin "14"
+		)
+		(pin "16"
+		)
+		(pin "7"
+		)
+		(pin "6"
+		)
+		(pin "24"
+		)
+		(pin "23"
+		)
+		(pin "21"
+		)
+		(pin "20"
+		)
+		(pin "19"
+		)
+		(instances
+			(project ""
+				(path "/cb36ad1e-370d-40ee-858e-c0dcf3346054"
+					(reference "U1")
+					(unit 1)
+				)
+			)
+		)
+	)
+	(symbol
 		(lib_id "power:GND")
 		(at 236.22 34.29 0)
@@
 		)
 	)
+	(embedded_fonts no)
 )

Commit message: new
Parts:
- added J2, J3, J4, J5, J6: Conn_01x04, symbol EESTN5:Conn_01x04
- added J7, J8: TB_1X2, symbol EESTN5:TB_1X2
- added R1, R10, R2, R3, R4, R5, R6, R7, R8, R9: R, symbol EESTN5:R
- added U2, U3: TA6586, symbol MacroLib:TA6586
Connections:
- net +5V: now also U1.18 (VIN), J2.2 (Pin_2), J3.2 (Pin_2), J4.2 (Pin_2), J5.2 (Pin_2), J6.2 (Pin_2)
- net D1: now also U1.7 (IO33)
- net D2: now also U1.6 (IO32)
- net D3: now also U1.5 (IO35)
- net D4: now also U1.4 (IO34)
- net D5: now also U1.3 (SENSOR_VN)
- net D6: now also U1.2 (SENSOR_VP)
- net D7: now also U1.36 (IO23)
- net D8: now also U1.35 (IO22)
- net GND: now also J2.1 (Pin_1), J3.1 (Pin_1), J4.1 (Pin_1), J5.1 (Pin_1), J6.1 (Pin_1), R10.2, R2.2, R4.2, R6.2, R8.2, U2.3 (GND), U3.3 (GND)
- net OUT_S3: now reaches U1.10 (IO27)
- net OUT_S3: now also R5.2, R6.1
- net OUT_S4: now reaches U1.11 (IO14)
- net OUT_S4: now also R7.2, R8.1
- net OUT_S5: now reaches U1.13 (IO13)
- net OUT_S5: now also R10.1, R9.2
- net OUT_S1: now reaches U1.8 (IO25)
- net OUT_S1: now also R1.2, R2.1
- net OUT_S2: now reaches U1.9 (IO26)
- net OUT_S2: now also R3.2, R4.1
- new net: J7.2, U2.5 (OUTF), U2.6 (OUTF)
- new net: J7.1, U2.7 (OUTR), U2.8 (OUTR)
- new net: J8.1, U3.7 (OUTR), U3.8 (OUTR)
- new net: J8.2, U3.5 (OUTF), U3.6 (OUTF)
- new net S1: J2.3 (Pin_3), R1.1
- new net S2: J3.3 (Pin_3), R3.1
- new net S3: J4.3 (Pin_3), R5.1
- new net S4: J5.3 (Pin_3), R7.1
- new net S5: J6.3 (Pin_3), R9.1
- new net VCC: U2.4 (VCC), U3.4 (VCC)
Other:
- moved on the sheet: J1

Commit message: new
Parts:
- added C1, C2, C3, C4: C, symbol EESTN5:C
- added J10, J11, J9: Conn_01X03, symbol EESTN5:Conn_01X03
Connections:
- net +3.3V: now also J10.1 (P1), J11.1 (P1), J9.1 (P1)
- net GND: now also C1.2, C2.2, C3.2, C4.2, J10.3 (P3), J11.3 (P3), J9.3 (P3)
- net VCC: now also C1.1, C2.1, C3.1, C4.1
- net T3: now reaches U1.26 (IO4)
- net T3: now also J11.2 (P2)
- net M2A: now reaches U1.27 (RX2)
- net M2A: now also U3.2 (INF)
- net M2B: now reaches U1.28 (TX2)
- net M2B: now also U3.1 (INR)
- net T2: now reaches U1.29 (IO5)
- net T2: now also J10.2 (P2)
- net T1: now reaches U1.30 (IO18)
- net T1: now also J9.2 (P2)
- net M1A: now reaches U1.31 (IO19)
- net M1A: now also U2.2 (INF)
- net M1B: now reaches U1.32 (IO21)
- net M1B: now also U2.1 (INR)
Other:
- moved on the sheet: J2, J3, J4, J5, J6, U1

Commit message: new
Parts:
- added IC1: CD4051B, CDIP762W66P254L2134H508Q16, symbol Logic_Gate:CD4051B
- added J12: Conn_01x04, symbol EESTN5:Conn_01x04
Connections:
- net +5V: now also IC1.16 (VDD), J12.4 (Pin_4)
- net D1: now also IC1.13 (CH_0); no longer U1.7 (IO33)
- net D2: now also IC1.14 (CH_1); no longer U1.6 (IO32)
- net D3: now also IC1.15 (CH_2); no longer U1.5 (IO35)
- net D4: now also IC1.12 (CH_3); no longer U1.4 (IO34)
- net D5: now also IC1.1 (CH_4); no longer U1.3 (SENSOR_VN)
- net D6: now also IC1.5 (CH_5); no longer U1.2 (SENSOR_VP)
- net D7: now also IC1.2 (CH_6); no longer U1.36 (IO23)
- net D8: now also IC1.4 (CH_7); no longer U1.35 (IO22)
- net GND: now also IC1.6 (INH), IC1.7 (VEE), IC1.8 (VSS), J12.1 (Pin_1)
- net M1A: now also U1.30 (IO18); no longer U1.31 (IO19)
- net M1B: now also U1.31 (IO19); no longer U1.32 (IO21)
- net T1: now also U1.29 (IO5); no longer U1.30 (IO18)
- net T2: now also U1.26 (IO4); no longer U1.29 (IO5)
- net T3: now also U1.24 (IO15); no longer U1.26 (IO4)
- new net COM: IC1.3 (COM), U1.2 (SENSOR_VP)
- new net INA: IC1.11 (A), U1.36 (IO23)
- new net INB: IC1.10 (B), U1.35 (IO22)
- new net INC: IC1.9 (C), U1.32 (IO21)
- new net SCL: J12.2 (Pin_2), U1.6 (IO32)
- new net SDA: J12.3 (Pin_3), U1.7 (IO33)

Commit message: new
Parts:
- added P1: CONN_01X08, symbol EESTN5:CONN_01X08
Connections:
- net +5V: now also P1.1 (P1)
- net GND: now also P1.2 (P2)
- net SCL: now also P1.3 (P3)
- net SDA: now also P1.4 (P4)
- new net INT: P1.8 (P8)
- no-connect marks 0 -> 3

Commit message: new
Parts:
- removed C1, C2, C3, C4: C, symbol EESTN5:C
- removed IC1: CD4051B, CDIP762W66P254L2134H508Q16, symbol Logic_Gate:CD4051B
- removed J7, J8: TB_1X2, symbol EESTN5:TB_1X2
- removed U1: ESP32_DevKit_V1_DOIT, ESP32_DevKit_V1_DOIT:esp32_devkit_v1_doit, symbol EESTN5:ESP32_DevKit_V1_DOIT
- removed U2, U3: TA6586, symbol MacroLib:TA6586
- added C1, C2, C3, C4, C5, C8, C9: C_Polarized, symbol Device:C_Polarized
- added C6, C7: C, symbol Device:C
- added D1: B340, Diode_SMD:D_SMC, symbol Diode:B340
- added IC1, IC2, IC3, IC4: BTS7960B, BTS7960B, symbol Mosfet:BTS7960B
- added L1, L2, L3: L, symbol Device:L
- added R11, R12: R, symbol EESTN5:R
- added SW1: SW_SPDT, symbol Switch:SW_SPDT
- added U1: LM2596S-5, Package_TO_SOT_SMD:TO-263-5_TabPin3, symbol Regulator_Switching:LM2596S-5
- added U4: ESP32-S3-WROOM-1, RF_Module:ESP32-S3-WROOM-1, symbol RF_Module:ESP32-S3-WROOM-1
- added U5: AMS1117-3.3, Package_TO_SOT_SMD:SOT-223-3_TabPin2, symbol Regulator_Linear:AMS1117-3.3
Connections:
- net GND: now also C1.2, C2.2, C3.2, C4.2, C5.2, C6.2, C7.2, C8.2, C9.2, D1.2 (A), IC1.1 (GND), IC2.1 (GND), IC3.1 (GND), IC4.1 (GND), R11.2, SW1.1 (A), U1.3 (GND), U5.1 (GND)
- net VCC: now also IC1.7 (VS), IC2.7 (VS), IC3.7 (VS), IC4.7 (VS)
- new net: D1.1 (K), L1.1, U1.2 (OUT)
- new net: C1.1, L1.2, L2.1, U1.4 (FB)
- new net: R11.1, R12.2, SW1.3 (C)
- new net: C2.1, C8.1, L3.2, R12.1, U1.1 (VIN)
- new net: SW1.2 (B), U1.5 (~{ON}/OFF)
- new net: C5.1, C7.1, U5.2 (VO)
- new net: U4.1 (GND), U4.40 (GND), U4.41 (GND)
- new net: C9.1, L3.1
- new net: C3.1, C4.1, C6.1, L2.2, U5.3 (VI)
Other:
- moved on the sheet: J1, J10, J11, J12, J2, J3, J4, J5, J6, J9, R1, R10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
